File: hv_supply.kicad_sch (KiCad schematic)
At the start: 0 parts

Commit message: built out power supplies, added datasheets
Parts:
- added C24: 100nF, Capacitor_SMD:C_0402_1005Metric, symbol Device:C
- added C25: 470pF, Capacitor_SMD:C_0402_1005Metric, symbol Device:C
- added C26, C27: 0, Capacitor_SMD:C_0402_1005Metric, symbol Device:C
- added C28: 4.7uF, Capacitor_SMD:C_0603_1608Metric, symbol Device:C
- added C29: 1uF, Capacitor_SMD:C_2220_5750Metric, symbol Device:C
- added C30: 100nF, Capacitor_SMD:C_2220_5750Metric, symbol Device:C
- added D1: STTH1R04AY, Diode_SMD:D_SMA, symbol Device:D
- added Q3: PSMN5R2-60YL, Package_TO_SOT_SMD:LFPAK56, symbol Transistor_FET:PSMN5R2-60YL
- added R23: 300k, Capacitor_SMD:C_0402_1005Metric, symbol Device:R_US
- added R24: 86.6k, Capacitor_SMD:C_0402_1005Metric, symbol Device:R_US
- added R25, R26: 0, Capacitor_SMD:C_0402_1005Metric, symbol Device:R_US
- added R27: 10m, Resistor_SMD:R_2512_6332Metric, symbol Device:R_US
- added R28: 1.5M, Resistor_SMD:R_1206_3216Metric, symbol Device:R_US
- added R29: 13.7k, Resistor_SMD:R_0603_1608Metric, symbol Device:R_US
- added T1: 750312367, symbol Device:750312367
- added U9: LT3757EDD, Package_DFN_QFN:DFN-10-1EP_3x3mm_P0.5mm_EP1.55x2.48mm, symbol Regulator_Switching:LT3757EDD
Connections:
- new net: R28.1, R29.2, U9.2 (FBX)
- new net: C28.1, U9.8 (INTVCC)
- new net: C26.1, R23.1, U9.1 (VC)
- new net: C24.1, U9.3 (SS)
- new net: R24.1, U9.4 (RT)
- new net: C27.1, R26.1, U9.6 (SENSE)
- new net: R25.1, U9.7 (GATE)
- new net: C25.1, R23.2
- new net: Q3.1 (S), Q3.2 (S), Q3.3 (S), R26.2, R27.2
- new net: Q3.4 (G), R25.2
- new net: D1.2 (A), T1.3 (SA)
- new net: Q3.5 (D), T1.4 (AB)
- new net GND: C24.2, C25.2, C26.2, C27.2, C28.2, C29.1, C30.1, R24.2, R27.1, R29.1, T1.1 (SB), U9.11 (GND), U9.5 (SYNC)
- new net HV_OUT: C29.2, C30.2, D1.1 (K), R28.2
- new net VBUS: T1.6 (AA), U9.10 (VIN)
