File: usb_pd.kicad_sch (KiCad schematic)
At the start: 10 parts, among them J1 USB_C_Receptacle, Q1 DMN3008SFG, Q2 DMN3008SFG, U7 AP33772

Commit message: built out power supplies, added datasheets
Connections:
- net VBUS: now reaches Q2.5 (D), R19.2
Changed lines of the file:
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@@
   (junction (at 97.79 85.09) (diameter 0) (color 0 0 0 0)
+  )
+  (junction (at 171.45 49.53) (diameter 0) (color 0 0 0 0)
   )
   (junction (at 90.17 87.63) (diameter 0) (color 0 0 0 0)
@@
     (stroke (width 0) (type default))
   )
+  (wire (pts (xy 171.45 49.53) (xy 176.53 49.53))
+    (stroke (width 0) (type default))
+  )
   (wire (pts (xy 171.45 49.53) (xy 166.37 49.53))
     (stroke (width 0) (type default))
@@
     (effects (font (size 1.27 1.27)) (justify left))
   )
+  (hierarchical_label "VBUS" (shape output) (at 176.53 49.53 0) (fields_autoplaced)
+    (effects (font (size 1.27 1.27)) (justify left))
+  )
